File: hardware/brdstepper/brdstepper.kicad_sch (KiCad schematic)
At the start: 0 parts

Commit message: brdstepper KiCad: the schematic on one large sheet
The five sheets (power, mcu, bridges, encoder, interfaces) become framed,
titled sections of one sheet, packed into columns on the smallest paper
that holds them (A2, two columns); pins join by net labels instead of
global labels. The netlist is unchanged (gen/check.py: 94 parts, 67
nets), the board regenerated with its footprints linked to the new
symbols, DRC clean but for the unrouted connections.

Co-Authored-By: Claude Opus 5.5 <noreply@anthropic.com>
Claude-Session: https://claude.ai/code/session_015Arx3mBYT6sxmWehm9yoEa
Parts:
- added C1, C2: 22u 50V, Capacitor_SMD:C_1210_3225Metric, symbol Device:C
- added C10, C12, C8, C9: 1u, Capacitor_SMD:C_0402_1005Metric, symbol Device:C
- added C11, C13, C14, C22, C36: 10n, Capacitor_SMD:C_0402_1005Metric, symbol Device:C
- added C15, C16: 10p C0G, Capacitor_SMD:C_0402_1005Metric, symbol Device:C
- added C17, C18, C19, C20, C33, C34, C38, C39, C40, C5: 100n, Capacitor_SMD:C_0402_1005Metric, symbol Device:C
- added C21: 4.7u, Capacitor_SMD:C_0603_1608Metric, symbol Device:C
- added C23, C27, C4: 100n 50V, Capacitor_SMD:C_0402_1005Metric, symbol Device:C
- added C24, C28: 10u 50V, Capacitor_SMD:C_1206_3216Metric, symbol Device:C
- added C25, C29: 100n 16V, Capacitor_SMD:C_0402_1005Metric, symbol Device:C
- added C26, C30: 22n 50V, Capacitor_SMD:C_0402_1005Metric, symbol Device:C
- added C3: 2.2u 50V, Capacitor_SMD:C_1206_3216Metric, symbol Device:C
- added C31, C32: 100p C0G, Capacitor_SMD:C_0402_1005Metric, symbol Device:C
- added C35: 10u, Capacitor_SMD:C_0603_1608Metric, symbol Device:C
- added C37: 4.7n, Capacitor_SMD:C_0402_1005Metric, symbol Device:C
- added C6, C7: 22u 10V, Capacitor_SMD:C_0805_2012Metric, symbol Device:C
- added D1: BAT54C, Package_TO_SOT_SMD:SOT-23, symbol Diode:BAT54C
- added D2: SMAJ24A, Diode_SMD:D_SMA, symbol Diode:SMAJ24A
- added D3, D5: BAT54WS, Diode_SMD:D_SOD-323, symbol Device:D_Schottky
- added D4: green, LED_SMD:LED_0603_1608Metric, symbol Device:LED
- added FB1: 600R@100MHz, Inductor_SMD:L_0603_1608Metric, symbol Device:FerriteBead_Small
- added H1, H2, H3, H4: M2.5, MountingHole:MountingHole_2.7mm_M2.5, symbol Mechanical:MountingHole
- added J1: USB-C, Connector_USB:USB_C_Receptacle_GCT_USB4105-xx-A_16P_TopMnt_Horizontal, symbol Connector:USB_C_Receptacle_USB2.0_16P
- added J2: VM / GND / EN, Connector_JST:JST_XH_B3B-XH-A_1x03_P2.50mm_Vertical, symbol Connector_Generic:Conn_01x03
- added J3: MOTOR, Connector_PinHeader_2.00mm:PinHeader_1x04_P2.00mm_Vertical, symbol Connector_Generic:Conn_01x04
- added J4: SMART-SERIAL, Connector_JST:JST_GH_SM06B-GHS-TB_1x06-1MP_P1.25mm_Horizontal, symbol Connector_Generic_MountingPin:Conn_01x06_MountingPin
- added J5, J6: CAN, Connector_JST:JST_GH_SM04B-GHS-TB_1x04-1MP_P1.25mm_Horizontal, symbol Connector_Generic_MountingPin:Conn_01x04_MountingPin
- added J7: SWD, Connector_PinHeader_1.27mm:PinHeader_1x05_P1.27mm_Vertical_SMD_Pin1Left, symbol Connector_Generic:Conn_01x05
- added JP1: TERM, Jumper:SolderJumper-2_P1.3mm_Open_RoundedPad1.0x1.5mm, symbol Jumper:SolderJumper_2_Open
- added L1: 10u, Inductor_SMD:L_Taiyo-Yuden_NR-40xx, symbol Device:L
- added R1: 88.7k 1%, Resistor_SMD:R_0402_1005Metric, symbol Device:R
- added R10, R4: 10k 1%, Resistor_SMD:R_0402_1005Metric, symbol Device:R
- added R11, R12: 2.0k 1%, Resistor_SMD:R_0402_1005Metric, symbol Device:R
- added R13, R16: 100k, Resistor_SMD:R_0402_1005Metric, symbol Device:R
- added R14, R15, R5, R7, R8: 10k, Resistor_SMD:R_0402_1005Metric, symbol Device:R
- added R17, R18: 5.1k, Resistor_SMD:R_0402_1005Metric, symbol Device:R
- added R19: 1M, Resistor_SMD:R_0402_1005Metric, symbol Device:R
- added R2: 22.1k 1%, Resistor_SMD:R_0402_1005Metric, symbol Device:R
- added R20, R21: 120, Resistor_SMD:R_0402_1005Metric, symbol Device:R
- added R3: 100k 1%, Resistor_SMD:R_0402_1005Metric, symbol Device:R
- added R6, R9: 1k, Resistor_SMD:R_0402_1005Metric, symbol Device:R
- added TH1: 10k B3380, Resistor_SMD:R_0603_1608Metric, symbol Device:Thermistor_NTC
- added TP1: AIN, TestPoint:TestPoint_Pad_D1.0mm, symbol Connector:TestPoint
- added TP2: PB10, TestPoint:TestPoint_Pad_D1.0mm, symbol Connector:TestPoint
- added TP3: PB11, TestPoint:TestPoint_Pad_D1.0mm, symbol Connector:TestPoint
- added U1: STM32G473CEU6, Package_DFN_QFN:QFN-48-1EP_7x7mm_P0.5mm_EP5.6x5.6mm, symbol MCU_ST_STM32G4:STM32G473CEUx
- added U2, U3: DRV8876RGTR, Package_DFN_QFN:VQFN-16-1EP_3x3mm_P0.5mm_EP1.68x1.68mm_ThermalVias, symbol brdstepper:DRV8876RGT
- added U4: AS5047P-ATSM, Package_SO:TSSOP-14_4.4x5mm_P0.65mm, symbol brdstepper:AS5047P
- added U5: TLV75533PDBVR, Package_TO_SOT_SMD:SOT-23-5, symbol Regulator_Linear:TLV75533PDBV
- added U6: TPS560430XDBVR, Package_TO_SOT_SMD:SOT-23-6, symbol brdstepper:TPS560430
- added U7: USBLC6-2SC6, Package_TO_SOT_SMD:SOT-23-6, symbol Power_Protection:USBLC6-2SC6
- added U8: SN65HVD30DR, Package_SO:SOIC-8_3.9x4.9mm_P1.27mm, symbol Interface_UART:MAX3490xSA
- added U9: TCAN1044VDR, Package_SO:SOIC-8_3.9x4.9mm_P1.27mm, symbol Interface_CAN_LIN:TJA1042T-3
- added Y1: 8MHz, Crystal:Crystal_SMD_2016-4Pin_2.0x1.6mm, symbol Device:Crystal_GND24
Connections:
- new net 3V3: C18.1, C19.1, C20.1, C21.1, C34.1, C35.1, C38.1, C40.1, C9.1, D5.1 (K), FB1.1, J7.1 (Pin_1), R10.1, R14.2, R7.1, U1.1 (VBAT), U1.23 (VDD), U1.35 (VDD), U1.48 (VDD), U2.14 (PMODE), U3.14 (PMODE), U4.11 (VDD), U4.12 (VDD3V3), U5.5 (OUT), U8.1 (VCC), U9.5 (VIO)
- new net 5V: C39.1, C8.1, D1.3, D3.1 (K), U5.1 (IN), U5.3 (EN), U9.3 (VCC)
- new net 5V_BUCK: C6.1, C7.1, D1.1, L1.2, R1.1
- new net 5V_MESA: D3.2 (A), J4.5 (Pin_5)
- new net 5V_USB: D1.2, J1.A4 (VBUS), J1.A9 (VBUS), J1.B4 (VBUS), J1.B9 (VBUS), U7.5 (VBUS)
- new net AIN: C22.1, R9.2, U1.17 (PB0)
- new net AIN_IN: R9.1, TP1.1
- new net A_IN1: U1.30 (PA8), U2.15 (EN/IN1)
- new net A_IN2: U1.31 (PA9), U2.16 (PH/IN2)
- new net BUCK_CB: C5.1, U6.1 (CB)
- new net BUCK_FB: R1.2, R2.1, U6.3 (FB)
- new net BUCK_SW: C5.2, L1.1, U6.6 (SW)
- new net B_IN1: U1.32 (PA10), U3.15 (EN/IN1)
- new net B_IN2: U1.29 (PC6), U3.16 (PH/IN2)
- new net CANH: J5.1 (Pin_1), J6.1 (Pin_1), JP1.1 (A), U9.7 (CANH)
- new net CANL: J5.2 (Pin_2), J6.2 (Pin_2), R21.2, U9.6 (CANL)
- new net CAN_RX: R5.1, U1.46 (PB8), U9.4 (RXD)
- new net CAN_STB: U1.26 (PB13), U9.8 (STB)
- new net CAN_TERM: JP1.2 (B), R21.1
- new net CAN_TX: U1.47 (PB9), U9.1 (TXD)
- new net COIL_A+: J3.1 (Pin_1), U2.6 (OUT1)
- new net COIL_A-: J3.2 (Pin_2), U2.8 (OUT2)
- new net COIL_B+: J3.3 (Pin_3), U3.6 (OUT1)
- new net COIL_B-: J3.4 (Pin_4), U3.8 (OUT2)
- new net ENC_CLK: U1.41 (PB3), U4.2 (CLK)
- new net ENC_CS: U1.38 (PA15), U4.1 (~{CS})
- new net ENC_MISO: U1.42 (PB4), U4.3 (MISO)
- new net ENC_MOSI: U1.43 (PB5), U4.4 (MOSI)
- new net EN_IN: C36.1, D5.2 (A), R15.2, R16.1, U1.15 (PA7)
- new net EN_RAW: J2.3 (Pin_3), R15.1
- new net GND: C1.2, C10.2, C11.2, C12.2, C13.2, C14.2, C15.2, C16.2, C17.2, C18.2, C19.2, C2.2, C20.2, C21.2, C22.2, C23.2, C24.2, C27.2, C28.2, C3.2, C31.2, C32.2, C33.2, C34.2, C35.2, C36.2, C37.2, C38.2, C39.2, C4.2, C40.2, C6.2, C7.2, C8.2, C9.2, D2.2 (A2), D4.1 (K), J1.A1 (GND), J1.A12 (GND), J1.B1 (GND), J1.B12 (GND), J2.2 (Pin_2), J4.6 (Pin_6), J4.MP (MountPin), J5.4 (Pin_4), J5.MP (MountPin), J6.4 (Pin_4), J6.MP (MountPin), J7.5 (Pin_5), R11.2, R12.2, R13.2, R16.2, R17.2, R18.2, R19.2, R2.2, R4.2, R5.2, R8.2, TH1.2, U1.49 (VSS), U2.13 (GND), U2.17 (PAD), U2.7 (PGND), U3.13 (GND), U3.17 (PAD), U3.7 (PGND), U4.13 (GND), U4.5 (TST), U5.2 (GND), U6.2 (GND), U7.2 (GND), U8.4 (GND), U9.2 (GND), Y1.2, Y1.4
- new net HWID: R7.2, R8.1, U1.18 (PB1)
- new net IPROPI_A: C31.1, R11.1, U1.8 (PA0), U2.4 (IPROPI)
- new net IPROPI_B: C32.1, R12.1, U1.9 (PA1), U3.4 (IPROPI)
- new net LED: R6.1, U1.25 (PB12)
- new net LED_A: D4.2 (A), R6.2
- new net NRST: C17.1, J7.3 (Pin_3), U1.7 (PG10)
- new net NTC: R10.2, TH1.1, U1.11 (PA3)
- new net OSC_IN: C15.1, U1.5 (PF0), Y1.1
- new net OSC_OUT: C16.1, U1.6 (PF1), Y1.3
- new net SS_RX: U1.45 (PB7), U8.2 (RO)
- new net SS_RX+: J4.3 (Pin_3), R20.1, U8.8 (A)
- new net SS_RX-: J4.4 (Pin_4), R20.2, U8.7 (B)
- new net SS_TX: U1.44 (PB6), U8.3 (DI)
- new net SS_TX+: J4.1 (Pin_1), U8.5 (Y)
- new net SS_TX-: J4.2 (Pin_2), U8.6 (Z)
- new net SWCLK: J7.4 (Pin_4), U1.37 (PA14)
- new net SWDIO: J7.2 (Pin_2), U1.36 (PA13)
- new net TP_PB10: TP2.1, U1.22 (PB10)
- new net TP_PB11: TP3.1, U1.24 (PB11)
- new net U2_CPH: C26.1, U2.11 (CPH)
- new net U2_CPL: C26.2, U2.12 (CPL)
- new net U2_VCP: C25.1, U2.10 (VCP)
- new net U3_CPH: C30.1, U3.11 (CPH)
- new net U3_CPL: C30.2, U3.12 (CPL)
- new net U3_VCP: C29.1, U3.10 (VCP)
- new net USB_CC1: J1.A5 (CC1), R17.1
- new net USB_CC2: J1.B5 (CC2), R18.1
- new net USB_DM: J1.A7 (D-), J1.B7 (D-), U1.33 (PA11), U7.1 (I/O1), U7.6 (I/O1)
- new net USB_DP: J1.A6 (D+), J1.B6 (D+), U1.34 (PA12), U7.3 (I/O2), U7.4 (I/O2)
- new net USB_SHIELD: C37.1, J1.S1 (SHIELD), R19.1
- new net VDDA: C10.1, C11.1, C12.1, C13.1, FB1.2, U1.20 (VREF+), U1.21 (VDDA)
- new net VM: C1.1, C2.1, C23.1, C24.1, C25.2, C27.1, C28.1, C29.2, C3.1, C4.1, D2.1 (A1), J2.1 (Pin_1), J5.3 (Pin_3), J6.3 (Pin_3), R3.1, U2.9 (VM), U3.9 (VM), U6.4 (EN), U6.5 (VIN)
- new net VM_SENSE: C14.1, R3.2, R4.1, U1.10 (PA2)
- new net VREF_DRV: C33.1, U1.12 (PA4), U2.3 (VREF), U3.3 (VREF)
- new net nFAULT: R14.1, U1.14 (PA6), U2.2 (nFAULT), U3.2 (nFAULT)
- new net nSLEEP: R13.1, U1.13 (PA5), U2.1 (nSLEEP), U3.1 (nSLEEP)
- no-connect marks 0 -> 19
Other:
- removed sheet bridges
- removed sheet encoder
- removed sheet interfaces
- removed sheet mcu
- removed sheet power
- note added: "brdstepper: STM32G473 + AS5047P + 2x DRV8876, 28 x 28 mm on the back of a NEMA11 motor. Connections are by net name (net labels): docs/brdstepper_hw.md is the reference. Variant A fits U8/J4 (smart-serial to a Mesa card), variant B U9/J5/J6/JP1 (CAN)."
- note removed: "brdstepper: STM32G473 + AS5047P + 2x DRV8876, 28 x 28 mm on the back of a NEMA11 motor. Connections are by net name (global labels): docs/brdstepper_hw.md is the reference. Variant A fits U8/J4 (smart-serial to a Mesa card), variant B U9/J5/J6/JP1 (CAN)."
