File: hardware/vibsensor/vibsensor.kicad_sch (KiCad schematic)
At the start: 50 parts, among them J1 M8 LEADS, J2 SWD, U1 STM32G473CEU6, U2 TPS560430XDBVR, U3 TLV75533PDBVR, U4 IIS3DWBTR, U5 TMP117AIDRVR, U6 TCAN1044VDR, Y1 8MHz

Commit message: vibsensor: two M8 sockets (IN / OUT) and a terminator plug
The sensors daisy-chain on standard M8 4-pin cables: IN (male) and OUT
(female), wired 1:1 on the board (J1, J3), so supply and CAN pass
through. The on-board termination (JP1, R10) is gone; the last sensor's
OUT takes an M8 male plug with the 120 ohm inside.

Enclosure: both sockets on the tail's 45-degree faces, the M4 lugs on
the X axis at the nose and tail, a terminated render. Docs updated.

Co-Authored-By: Claude Opus 5.5 <noreply@anthropic.com>
Claude-Session: https://claude.ai/code/session_015Arx3mBYT6sxmWehm9yoEa
Parts:
- removed JP1: TERM, Jumper:SolderJumper-2_P1.3mm_Open_RoundedPad1.0x1.5mm, symbol Jumper:SolderJumper_2_Open
- removed R10: 120, Resistor_SMD:R_0402_1005Metric, symbol Device:R
- added J3: M8 OUT, Connector_PinHeader_2.00mm:PinHeader_1x04_P2.00mm_Vertical, symbol Connector_Generic:Conn_01x04
- J1: value M8 LEADS -> M8 IN; Note the M8 socket's leads, M8 order: 1 V+, 2 CAN_H, 3 GND, 4 CA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 -> the IN socket's leads (M8 male), M8 order: 1 V+, 2 CAN_H, 3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
Connections:
- net 24V_IN: now also J3.1 (Pin_1)
- net CANH: now also J3.2 (Pin_2)
- net CANL: now also J3.4 (Pin_4)
- net GND: now also J3.3 (Pin_3)
Other:
- note added: "CAN FD transceiver, mounting (termination: a plug in the last sensor's OUT)"
- note added: "Supply: M8 IN / OUT (passed through), reverse polarity, TVS, buck 5 V, LDO 3.3 V, filtered rails, bus voltage"
- note added: "vibsensor: STM32G473 + IIS3DWB + TMP117 + TCAN1044V on a round board, potted in the sensor's housing. Two M8 4-pin sockets (1 V+, 2 CAN_H, 3 GND, 4 CAN_L): IN (J1) and OUT (J3), the bus and supply passed through; the last sensor's OUT takes a terminator plug (120 ohm). Node number and name over the bus (no jumpers). Connections are by net name (net labels): docs/vibsensor.md and vibsensor/inc/vs.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"
- note removed: "CAN FD transceiver, termination, mounting"
- note removed: "Supply: reverse polarity, TVS, buck 5 V, LDO 3.3 V, filtered rails, bus voltage"
- note removed: "vibsensor: STM32G473 + IIS3DWB + TMP117 + TCAN1044V on a round board, potted in the sensor's housing. M8 4-pin (1 V+, 2 CAN_H, 3 GND, 4 CAN_L) soldered to J1. Node number and name over the bus (no jumpers). Connections are by net name (net labels): docs/vibsensor.md and vibsensor/inc/vs.h are the reference."
- moved on the sheet: C1, C17, C18, C19, C2, C20, C3, C4, C5, C6, C7, C8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
